File: K8400-extboard.kicad_pcb (KiCad board)
At the start: 2 copper layers, 60 x 60 mm, 17 parts, among them J1 Part-2, J2 HEAT1, J3 RemoteHeader_10, J4 HEAT2, J5 Cool-1

Commit message: Smaller board Polazrized capacitor through the hole smaller LEDs
Parts:
- C1: footprint Capacitor_SMD:C_2010_5025Metric -> Capacitor_THT:CP_Radial_D5.0mm_P2.50mm; moved to F.Cu
- D2, D3: footprint Diode_SMD:D_SMA-SMB_Universal_Handsoldering -> LED_SMD:LED_1206_3216Metric
- moved J4 6.73 mm to (125.2, 97.0)
- moved J2 6.25 mm to (175.0, 90.0)
- moved D2 5.73 mm to (125.2, 105.8)
- moved D3 5.35 mm to (175.0, 107.9)
- moved R3 5.04 mm to (174.8, 116.7)
- moved R1 4.97 mm to (125.0, 114.9)
- moved C1 1.08 mm to (123.7, 81.3), turned to 90 degrees
- moved R2 0.80 mm to (125.1, 84.8), turned to 0 degrees
Routing:
- net /FAN+: track 32.5 -> 22.9 mm
- net /FAN-: track 26.1 -> 23.3 mm
- net Net-(C1-Pad1): track 13.7 -> 15.8 mm
Other:
- board size 60 x 60 mm -> 60 x 55 mm

Commit message: Wired
Parts:
- removed the R2 at (125.1, 84.8)
- added R3: 22, Resistor_SMD:R_1206_3216Metric, B.Cu at (124.6, 111.0)
- D3: renamed from D1; moved to B.Cu
- D4: moved to B.Cu
- moved R2 59.3 mm to (124.1, 85.9), turned to 180 degrees
- moved R1 59.1 mm to (176.1, 85.3), turned to 0 degrees
- moved D2 54.4 mm to (124.0, 89.2), turned to 0 degrees
- moved D1 53.7 mm to (176.1, 88.6), turned to 180 degrees
- moved C1 24.9 mm to (124.5, 106.2)
- moved J1 23.4 mm to (123.2, 96.8)
- moved D3 23.3 mm to (176.8, 106.2)
- moved D4 23.2 mm to (173.2, 106.0)
- moved J4 23.1 mm to (124.0, 74.0), turned to 270 degrees
- moved J5 22.6 mm to (173.7, 96.0)
- moved J2 9.06 mm to (176.0, 81.0), turned to 90 degrees
- moved J3 2.02 mm to (138.3, 72.0)
- renumbered D2 to D1, D3 to D2, R3 to R2
Connections:
- J2 pad 1: /HEAT1-B -> /TEMP1-A
- J2 pad 2: /HEAT1-A -> /TEMP1-B
- J2 pad 3: /TEMP1-B -> /HEAT1-A
- J2 pad 4: /TEMP1-A -> /HEAT1-B
- J4 pad 1: /TEMP2-B -> /HEAT2-A
- J4 pad 2: /TEMP2-A -> /HEAT1-B
- J4 pad 3: /HEAT1-B -> /TEMP2-A
- J4 pad 4: /HEAT2-A -> /TEMP2-B
Routing:
- net /HEAT1-B: track 0.00 -> 137.8 mm, vias 0 -> 2
- net /HEAT2-A: track 0.00 -> 102.4 mm, vias 0 -> 1
- net /HEAT1-A: track 0.00 -> 83.9 mm, vias 0 -> 1
- net /TEMP2-B: track 0.00 -> 36.9 mm, vias 0 -> 1
- net /TEMP2-A: track 0.00 -> 34.6 mm, vias 0 -> 1
- net /TEMP1-A: track 0.00 -> 33.7 mm, vias 0 -> 1
- net /TEMP1-B: track 0.00 -> 30.3 mm, vias 0 -> 1
- net /FAN+: track 22.9 -> 52.0 mm
- net /FAN-: track 23.3 -> 44.3 mm
- net Net-(D3-Pad1): track 0.00 -> 12.5 mm
- net Net-(D2-Pad2): track 0.00 -> 3.56 mm
- net Net-(D1-Pad2): track 0.00 -> 3.30 mm
Other:
- outline, holes or cut-outs redrawn
