File: K8400-extboard.sch (KiCad schematic (older format))
At the start: 13 parts, among them J1 Part-2, J2 HEAT1, J3 RemoteHeader_10, J4 HEAT2, J5 Cool-1

Commit message: Smaller board Polazrized capacitor through the hole smaller LEDs
Parts:
- C1: footprint Capacitor_SMD:C_2010_5025Metric -> Capacitor_THT:CP_Radial_D5.0mm_P2.50mm
- D2, D3: footprint Diode_SMD:D_SMA-SMB_Universal_Handsoldering -> LED_SMD:LED_1206_3216Metric
Changed lines of the file:
@@
 EESchema Schematic File Version 4
-LIBS:K8400-extboard-cache
-EELAYER 29 0
+EELAYER 30 0
 EELAYER END
 $Descr A4 11693 8268
@@
 F 0 "C1" H 3918 5446 50  0000 L CNN
 F 1 "22uF 50V" H 3918 5355 50  0000 L CNN
-F 2 "Capacitor_SMD:C_2010_5025Metric" H 3838 5250 50  0001 C CNN
+F 2 "Capacitor_THT:CP_Radial_D5.0mm_P2.50mm" H 3838 5250 50  0001 C CNN
 F 3 "~" H 3800 5400 50  0001 C CNN
 	1    3800 5400
@@
 F 0 "D2" V 3939 3733 50  0000 R CNN
 F 1 "LED" V 3848 3733 50  0000 R CNN
-F 2 "Diode_SMD:D_SMA-SMB_Universal_Handsoldering" H 3900 3850 50  0001 C CNN
+F 2 "LED_SMD:LED_1206_3216Metric" H 3900 3850 50  0001 C CNN
 F 3 "~" H 3900 3850 50  0001 C CNN
 	1    3900 3850
@@
 F 0 "D3" V 7639 3783 50  0000 R CNN
 F 1 "LED" V 7548 3783 50  0000 R CNN
-F 2 "Diode_SMD:D_SMA-SMB_Universal_Handsoldering" H 7600 3900 50  0001 C CNN
+F 2 "LED_SMD:LED_1206_3216Metric" H 7600 3900 50  0001 C CNN
 F 3 "~" H 7600 3900 50  0001 C CNN
 	1    7600 3900

Commit message: Wired
Parts:
- renumbered D2 to D1, D3 to D2, D1 to D3, R3 to R2, R2 to R3
Connections:
- net HEAT1-A: now also J2.3 (Pin_3); no longer J2.2 (Pin_2)
- net HEAT1-B: now also J2.4 (Pin_4), J4.2 (Pin_2); no longer J2.1 (Pin_1), J4.3 (Pin_3)
- net HEAT2-A: now also J4.1 (Pin_1); no longer J4.4 (Pin_4)
- net TEMP1-A: now also J2.1 (Pin_1); no longer J2.4 (Pin_4)
- net TEMP1-B: now also J2.2 (Pin_2); no longer J2.3 (Pin_3)
- net TEMP2-A: now also J4.3 (Pin_3); no longer J4.2 (Pin_2)
- net TEMP2-B: now also J4.4 (Pin_4); no longer J4.1 (Pin_1)
Changed lines of the file:
@@
 $EndComp
 $Comp
-L Device:R R3
+L Device:R R2
 U 1 1 5E8A16E9
 P 7900 3900
-F 0 "R3" H 7970 3946 50  0000 L CNN
+F 0 "R2" H 7970 3946 50  0000 L CNN
 F 1 "680" H 7970 3855 50  0000 L CNN
 F 2 "Resistor_SMD:R_1206_3216Metric" V 7830 3900 50  0001 C CNN
@@
 $EndComp
 $Comp
-L Device:R R2
+L Device:R R3
 U 1 1 5E8A1D6A
 P 4350 5350
-F 0 "R2" H 4420 5396 50  0000 L CNN
+F 0 "R3" H 4420 5396 50  0000 L CNN
 F 1 "22" H 4420 5305 50  0000 L CNN
 F 2 "Resistor_SMD:R_1206_3216Metric" V 4280 5350 50  0001 C CNN
@@
 $EndComp
 $Comp
-L Device:LED D2
+L Device:LED D1
 U 1 1 5E8A291F
 P 3900 3850
-F 0 "D2" V 3939 3733 50  0000 R CNN
+F 0 "D1" V 3939 3733 50  0000 R CNN
 F 1 "LED" V 3848 3733 50  0000 R CNN
 F 2 "LED_SMD:LED_1206_3216Metric" H 3900 3850 50  0001 C CNN
@@
 $EndComp
 $Comp
-L Device:LED D3
+L Device:LED D2
 U 1 1 5E8A3941
 P 7600 3900
-F 0 "D3" V 7639 3783 50  0000 R CNN
+F 0 "D2" V 7639 3783 50  0000 R CNN
 F 1 "LED" V 7548 3783 50  0000 R CNN
 F 2 "LED_SMD:LED_1206_3216Metric" H 7600 3900 50  0001 C CNN
@@
 FAN+
 $Comp
-L Diode:1N4148W D1
+L Diode:1N4148W D3
 U 1 1 5E90DADB
 P 2900 3850
-F 0 "D1" V 2946 3770 50  0000 R CNN
+F 0 "D3" V 2946 3770 50  0000 R CNN
 F 1 "1N4148W" V 2855 3770 50  0000 R CNN
 F 2 "Diode_SMD:D_SOD-123" H 2900 3675 50  0001 C CNN
@@
 L Connector:Conn_01x04_Female J2
 U 1 1 5E93778F
-P 4850 3150
-F 0 "J2" V 4788 2862 50  0000 R CNN
-F 1 "HEAT1" V 4697 2862 50  0000 R CNN
-F 2 "Connector_Molex:Molex_KK-254_AE-6410-04A_1x04_P2.54mm_Vertical" H 4850 3150 50  0001 C CNN
-F 3 "~" H 4850 3150 50  0001 C CNN
-	1    4850 3150
-	0    -1   -1   0
+P 4950 3150
+F 0 "J2" V 4888 2862 50  0000 R CNN
+F 1 "HEAT1" V 4797 2862 50  0000 R CNN
+F 2 "Connector_Molex:Molex_KK-254_AE-6410-04A_1x04_P2.54mm_Vertical" H 4950 3150 50  0001 C CNN
+F 3 "~" H 4950 3150 50  0001 C CNN
+	1    4950 3150
+	0    1    -1   0
 $EndComp
 $Comp
 L Connector:Conn_01x04_Female J4
 U 1 1 5E93AC82
-P 6200 3200
-F 0 "J4" V 6138 2912 50  0000 R CNN
-F 1 "HEAT2" V 6047 2912 50  0000 R CNN
-F 2 "Connector_Molex:Molex_KK-254_AE-6410-04A_1x04_P2.54mm_Vertical" H 6200 3200 50  0001 C CNN
-F 3 "~" H 6200 3200 50  0001 C CNN
-	1    6200 3200
-	0    -1   -1   0
-$EndComp
-Wire Wire Line
+P 6300 3200
+F 0 "J4" V 6238 2912 50  0000 R CNN
+F 1 "HEAT2" V 6147 2912 50  0000 R CNN
+F 2 "Connector_Molex:Molex_KK-254_AE-6410-04A_1x04_P2.54mm_Vertical" H 6300 3200 50  0001 C CNN
+F 3 "~" H 6300 3200 50  0001 C CNN
+	1    6300 3200
+	0    1    -1   0
+$EndComp
+Wire Wire Line
